File: drone/drone.kicad_pcb (KiCad board)
At the start: 2 copper layers, 81 x 70.3 mm, 12 parts, among them U2 ESP32-DEVKIT-V1

Commit message: Fixed PCB
Parts:
- removed ESC1, ESC2, ESC3: ~, Connector_PinSocket_2.54mm:PinSocket_1x02_P2.54mm_Vertical
- removed ESC4: ~, Connector_PinSocket_2.54mm:PinSocket_1x03_P2.54mm_Vertical
- removed the REF** at (170.8, 51.8)
- removed the REF** at (167.2, 80.3)
- added L1: ~, Connector_PinSocket_2.54mm:PinSocket_1x04_P2.54mm_Vertical, F.Cu at (157.6, 80.7)
- added REF**: PinSocket_1x06_P2.54mm_Vertical, Connector_PinSocket_2.54mm:PinSocket_1x06_P2.54mm_Vertical, F.Cu at (150.7, 74.4)
- added U3: ~, Connector_PinSocket_2.54mm:PinSocket_1x02_P2.54mm_Vertical, F.Cu at (152.0, 94.5)
- added U4: ~, Connector_PinSocket_2.54mm:PinSocket_1x02_P2.54mm_Vertical, F.Cu at (156.1, 94.5)
- added U5: ~, Connector_PinSocket_2.54mm:PinSocket_1x03_P2.54mm_Vertical, F.Cu at (160.3, 92.1)
- added U6: ~, Connector_PinSocket_2.54mm:PinSocket_1x04_P2.54mm_Vertical, F.Cu at (150.7, 64.3)
- added U7: ~, Connector_PinSocket_2.54mm:PinSocket_1x03_P2.54mm_Vertical, F.Cu at (167.4, 80.3)
- U1: value ~ -> ESP32-DEVKIT-V1; footprint Connector_PinSocket_2.54mm:PinSocket_1x10_P2.54mm_Vertical -> ESP32:MODULE_ESP32_DEVKIT_V1
- U2: value ESP32-DEVKIT-V1 -> ~; footprint esp32:MODULE_ESP32_DEVKIT_V1 -> Connector_PinSocket_2.54mm:PinSocket_1x02_P2.54mm_Vertical
- moved U2 27.4 mm to (147.8, 94.9), turned to 0 degrees
- moved U1 25.5 mm to (128.5, 75.5), turned to 180 degrees
Connections:
- U1 pad 1: 3V -> +3.3V
- U1 pad 10: (no net) -> unconnected-(U1-D19-Pad10)
- U1 pad 3: Net-(U1-SCL) -> unconnected-(U1-D15-Pad3)
- U1 pad 4: Net-(U1-SDA) -> unconnected-(U1-D2-Pad4)
- U1 pad 5: (no net) -> LED
- U1 pad 6: (no net) -> Net-(L1-TX)
- U1 pad 7: (no net) -> Net-(L1-RX)
- U1 pad 8: (no net) -> unconnected-(U1-D5-Pad8)
- U1 pad 9: (no net) -> unconnected-(U1-D18-Pad9)
- U2 pad 1: 3V -> PWM1
- U2 pad 2: (no net) -> GND
Routing:
- net Net-(ESC1-PWM): track 128.2 -> 0.00 mm
- net PWM4: track 0.00 -> 107.3 mm
- net PWM3: track 0.00 -> 93.4 mm
- net Net-(ESC4-PWM): track 83.2 -> 0.00 mm
- net 3V: track 77.9 -> 0.00 mm
- net Tx: track 62.0 -> 0.00 mm
- net 5Vin: track 61.3 -> 0.00 mm
- net +5V: track 0.00 -> 61.2 mm
- net Rx: track 59.6 -> 0.00 mm
- net PWM2: track 0.00 -> 48.9 mm
- net Net-(ESC3-PWM): track 47.1 -> 0.00 mm
- net +3.3V: track 0.00 -> 41.6 mm
- net Net-(U1-SDA): track 37.7 -> 0.00 mm
- net PWM1: track 0.00 -> 36.8 mm
- net Net-(L1-RX): track 0.00 -> 22.9 mm
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